File: shio.sch (KiCad schematic (older format))
At the start: 85 parts, among them J1 USB_B_Micro, U1 LM66100DCKT, U2 MAX38640AENT+, U3 NRF52840-CKAA-R7, U4 LM66100DCKT, U5 BMA400, U6 W25N01GVZEIG_TR, Y1 32.768kHz, Y2 32MHz

Commit message: All parts have associated components
Parts:
- BAT1: footprint (none) -> Shio:CR1632-THRU
- J1: footprint (none) -> digikey-footprints:USB_Micro_B_Female_10118193-0001LF
- MK1: footprint maruchi-kicad-library:MIC_ICS-41350 -> Shio:MIC_ICS-41350
- R10, R11, R6, R7: footprint Resistor_SMD:R_0201_0603Metric -> Resistor_SMD:R_0402_1005Metric
- U1, U4: footprint DCK6 -> Shio:LM66100DCKT
- U2: footprint 21-100128A_6_MXM -> Shio:MAX38640AENT&plus_
- U3: footprint maruchi-kicad-library:BGA94N35P10X10_360X354X51N -> Shio:BGA94N35P10X10_360X354X51N
- U5: footprint maruchi-kicad-library:XDCR_BMA400 -> Shio:XDCR_BMA400
- U6: footprint maruchi-kicad-library:SON127P800X600X80-9N -> Shio:SON127P800X600X80-9N
- Y1: footprint (none) -> Crystal:Crystal_SMD_3215-2Pin_3.2x1.5mm
Changed lines of the file:
@@
 F 0 "BAT1" H 9768 2996 50  0000 L CNN
 F 1 "1.8V-3.6V" H 9768 2905 50  0000 L CNN
-F 2 "" V 9650 2960 50  0001 C CNN
+F 2 "Shio:CR1632-THRU" V 9650 2960 50  0001 C CNN
 F 3 "~" V 9650 2960 50  0001 C CNN
 	1    9650 2900
@@
 F 0 "U6" H 8800 6520 50  0000 C CNN
 F 1 "W25N01GVZEIG_TR" H 8800 6429 50  0000 C CNN
-F 2 "maruchi-kicad-library:SON127P800X600X80-9N" H 8800 5850 50  0001 L BNN
+F 2 "Shio:SON127P800X600X80-9N" H 8800 5850 50  0001 L BNN
 F 3 "None" H 8800 5850 50  0001 L BNN
 F 4 "W25N01GVZEIG TR" H 8800 5850 50  0001 L BNN "Field4"
@@
 F 0 "J1" H 10507 3267 50  0000 C CNN
 F 1 "USB_B_Micro" H 10507 3176 50  0000 C CNN
-F 2 "" H 10600 2750 50  0001 C CNN
+F 2 "digikey-footprints:USB_Micro_B_Female_10118193-0001LF" H 10600 2750 50  0001 C CNN
 F 3 "~" H 10600 2750 50  0001 C CNN
 	1    10450 2800
@@
 F 0 "MK1" H 7700 4917 50  0000 C CNN
 F 1 "ICS-41350" H 7700 4826 50  0000 C CNN
-F 2 "maruchi-kicad-library:MIC_ICS-41350" H 7700 4450 50  0001 L BNN
+F 2 "Shio:MIC_ICS-41350" H 7700 4450 50  0001 L BNN
 F 3 "LGA-5 TDK-InvenSense" H 7700 4450 50  0001 L BNN
 F 4 "Bottom Port PDM Low Power muti-Mode Microphone with high AOP Mode" H 7700 4450 50  0001 L BNN "Field4"
@@
 F 0 "U3" H 2200 7317 50  0000 C CNN
 F 1 "NRF52840-CKAA-R7" H 2200 7226 50  0000 C CNN
-F 2 "maruchi-kicad-library:BGA94N35P10X10_360X354X51N" H 2200 7050 50  0001 L BNN
+F 2 "Shio:BGA94N35P10X10_360X354X51N" H 2200 7050 50  0001 L BNN
 F 3 "1.1" H 2200 7050 50  0001 L BNN
 F 4 "Nordic" H 2200 7050 50  0001 L BNN "Field4"
@@
 F 0 "R10" V 7795 2950 50  0000 C CNN
 F 1 "NC" V 7886 2950 50  0000 C CNN
-F 2 "Resistor_SMD:R_0201_0603Metric" H 8000 2950 50  0001 C CNN
+F 2 "Resistor_SMD:R_0402_1005Metric" H 8000 2950 50  0001 C CNN
 F 3 "~" H 8000 2950 50  0001 C CNN
 	1    8000 2950
@@
 F 0 "R11" V 8745 2950 50  0000 C CNN
 F 1 "NC" V 8836 2950 50  0000 C CNN
-F 2 "Resistor_SMD:R_0201_0603Metric" H 8950 2950 50  0001 C CNN
+F 2 "Resistor_SMD:R_0402_1005Metric" H 8950 2950 50  0001 C CNN
 F 3 "~" H 8950 2950 50  0001 C CNN
 	1    8950 2950
@@
 F 0 "U3" H 3050 6617 50  0000 C CNN
 F 1 "NRF52840-CKAA-R7" H 3050 6526 50  0000 C CNN
-F 2 "maruchi-kicad-library:BGA94N35P10X10_360X354X51N" H 3050 5050 50  0001 L BNN
+F 2 "Shio:BGA94N35P10X10_360X354X51N" H 3050 5050 50  0001 L BNN
 F 3 "1.1" H 3050 5050 50  0001 L BNN
 F 4 "Nordic" H 3050 5050 50  0001 L BNN "Field4"
@@
 F 0 "Y1" V 4096 6962 50  0000 R CNN
 F 1 "32.768kHz" V 4005 6962 50  0000 R CNN
-F 2 "" H 4050 7050 50  0001 C CNN
+F 2 "Crystal:Crystal_SMD_3215-2Pin_3.2x1.5mm" H 4050 7050 50  0001 C CNN
 F 3 "~" H 4050 7050 50  0001 C CNN
 	1    4050 7050
@@
 F 0 "U1" H 6450 1587 60  0000 C CNN
 F 1 "LM66100DCKT" H 6450 1481 60  0000 C CNN
-F 2 "DCK6" H 6450 1440 60  0001 C CNN
+F 2 "Shio:LM66100DCKT" H 6450 1440 60  0001 C CNN
 F 3 "" H 5650 1200 60  0000 C CNN
 	1    5650 1200
@@
 F 0 "U4" H 6450 2787 60  0000 C CNN
 F 1 "LM66100DCKT" H 6450 2681 60  0000 C CNN
-F 2 "DCK6" H 6450 2640 60  0001 C CNN
+F 2 "Shio:LM66100DCKT" H 6450 2640 60  0001 C CNN
 F 3 "" H 5650 2400 60  0000 C CNN
 	1    5650 2400
@@
 F 0 "U2" H 8850 1587 60  0000 C CNN
 F 1 "MAX38640AENT+" H 8850 1481 60  0000 C CNN
-F 2 "21-100128A_6_MXM" H 8850 1440 60  0001 C CNN
+F 2 "Shio:MAX38640AENT&plus_" H 8850 1440 60  0001 C CNN
 F 3 "" H 7950 1200 60  0000 C CNN
 	1    7950 1200
@@
 F 0 "R6" V 7795 2600 50  0000 C CNN
 F 1 "0R" V 7886 2600 50  0000 C CNN
-F 2 "Resistor_SMD:R_0201_0603Metric" H 8000 2600 50  0001 C CNN
+F 2 "Resistor_SMD:R_0402_1005Metric" H 8000 2600 50  0001 C CNN
 F 3 "~" H 8000 2600 50  0001 C CNN
 	1    8000 2600
@@
 F 0 "R7" V 8745 2600 50  0000 C CNN
 F 1 "0R" V 8836 2600 50  0000 C CNN
-F 2 "Resistor_SMD:R_0201_0603Metric" H 8950 2600 50  0001 C CNN
+F 2 "Resistor_SMD:R_0402_1005Metric" H 8950 2600 50  0001 C CNN
 F 3 "~" H 8950 2600 50  0001 C CNN
 	1    8950 2600
@@
 F 0 "U5" H 9900 5117 50  0000 C CNN
 F 1 "BMA400" H 9900 5026 50  0000 C CNN
-F 2 "maruchi-kicad-library:XDCR_BMA400" H 9900 4350 50  0001 L BNN
+F 2 "Shio:XDCR_BMA400" H 9900 4350 50  0001 L BNN
 F 3 "BMA400" H 9900 4350 50  0001 L BNN
 F 4 "LGA-12 Bosch Tools" H 9900 4350 50  0001 L BNN "Field4"
@@
 F 0 "U3" H 2900 2267 50  0000 C CNN
 F 1 "NRF52840-CKAA-R7" H 2900 2176 50  0000 C CNN
-F 2 "maruchi-kicad-library:BGA94N35P10X10_360X354X51N" H 2900 1600 50  0001 L BNN
+F 2 "Shio:BGA94N35P10X10_360X354X51N" H 2900 1600 50  0001 L BNN
 F 3 "1.1" H 2900 1600 50  0001 L BNN
 F 4 "Nordic" H 2900 1600 50  0001 L BNN "Field4"
